Commit message: hardware fix

File: scara_description/urdf/arm.xacro (robot description, xacro)
@@ -158,5 +158,5 @@
         <child link="wrist_link"/>
         <axis xyz="0 0 1"/>
-        <limit lower="-2.0" upper="2.0" effort="10.0" velocity="1.5"/>
+        <limit lower="-4.712" upper="4.712" effort="10.0" velocity="1.5"/>
     </joint>
     <!-- Tool centre point: centre of the gripper finger tips. -->

File: scara_description/urdf/ros2control.xacro (robot description, xacro)
@@ -81,6 +81,6 @@
         <joint name="wrist_joint">
             <command_interface name="position">
-                <param name="min">-2.0</param>
-                <param name="max">2.0</param>
+                <param name="min">-4.712</param>
+                <param name="max">4.712</param>
             </command_interface>
             <state_interface name="position"/>
